File: fc-nes.sch (EAGLE design)
At the start: 83 parts, among them X1 P1-PEG, X2 P2-PEG, X3 PEG-EXP

Commit message: .
Other:
- note added: "(DD14)"
- note added: "(DD6,DD7)"
- note added: "Питание"
- note added: "Тактовые генераторы"
