File: reversator/reversator.brd (EAGLE design)
At the start: 6 parts

Commit message: .
Parts:
- moved SLOT_N 21.0 mm to (0.64, 40.0)
- moved SLOT_F 15.2 mm to (0.00, 15.2)
- moved C60 15.2 mm to (0.00, 24.1)
- moved JP1 15.2 mm to (0.00, 21.0)
- moved C72 14.0 mm to (0.00, 26.7)
Routing:
- net GND: track 132.6 -> 182.4 mm
- net PA11: track 7.14 -> 33.0 mm
- net M2: track 6.50 -> 30.1 mm
- net D2: track 6.61 -> 29.5 mm
- net D5: track 6.61 -> 29.1 mm
- net D3: track 6.61 -> 28.7 mm
- net D1: track 6.61 -> 28.7 mm
- net D7: track 6.61 -> 28.5 mm
- net D6: track 6.61 -> 28.5 mm
- net A14: track 6.61 -> 28.5 mm
- net A13: track 6.61 -> 28.5 mm
- net A12: track 6.61 -> 28.5 mm
- net D0: track 6.61 -> 28.3 mm
- net D4: track 6.61 -> 28.0 mm
- net !ROMSEL: track 6.61 -> 27.6 mm
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
Commit message: 2
Parts:
- added U$1: 1X8, headers(2mm):1X8
Changed lines of the file:
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@@
 <board>
 <plain>
-<dimension x1="-45.72" y1="36.195" x2="-39.37" y2="19.05" x3="-53.975" y3="27.6225" textsize="1.778" layer="21" dtype="vertical"/>
+<dimension x1="-45.72" y1="36.195" x2="-40.64" y2="19.05" x3="-53.975" y3="27.6225" textsize="1.778" layer="21" dtype="vertical"/>
 <dimension x1="-167.64" y1="-1.905" x2="17.12595" y2="32.3723" x3="-75.257025" y3="103.505" textsize="1.778" layer="21" dtype="horizontal"/>
+<dimension x1="-34.29" y1="15.875" x2="36.83" y2="8.89" x3="1.27" y3="0.635" textsize="1.778" layer="1" dtype="horizontal"/>
 </plain>
 <attributes>
@@
 <element name="C72" library="h1,27mm" package="1X54" value="1X54" x="0" y="26.67"/>
 <element name="C60" library="h1,27mm" package="1X54" value="1X54" x="0" y="24.13"/>
+<element name="U$1" library="headers(2mm)" package="1X8" value="1X8" x="-159.385" y="-31.75"/>
 </elements>
 <signals>

Commit message: .
Parts:
- removed U$1: 1X8, headers(2mm):1X8
- added JP2, JP3, JP4, JP5: (no value), Разъёмы штырьковые 2.54мм:2X14
Changed lines of the file:
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@@
 <dimension x1="-167.64" y1="-1.905" x2="17.12595" y2="32.3723" x3="-75.257025" y3="103.505" textsize="1.778" layer="21" dtype="horizontal"/>
 <dimension x1="-34.29" y1="15.875" x2="36.83" y2="8.89" x3="1.27" y3="0.635" textsize="1.778" layer="1" dtype="horizontal"/>
+<dimension x1="-46.355" y1="45.72" x2="-48.26" y2="10.795" x3="-62.865" y3="28.2575" textsize="1.778" layer="21" dtype="vertical"/>
 </plain>
 <attributes>
@@
 <element name="C72" library="h1,27mm" package="1X54" value="1X54" x="0" y="26.67"/>
 <element name="C60" library="h1,27mm" package="1X54" value="1X54" x="0" y="24.13"/>
-<element name="U$1" library="headers(2mm)" package="1X8" value="1X8" x="-159.385" y="-31.75"/>
+<element name="JP2" library="Разъёмы штырьковые 2.54мм" package="2X14" value="" x="-88.265" y="43.815"/>
+<element name="JP3" library="Разъёмы штырьковые 2.54мм" package="2X14" value="" x="-120.65" y="32.385"/>
+<element name="JP4" library="Разъёмы штырьковые 2.54мм" package="2X14" value="" x="-120.65" y="24.765"/>
+<element name="JP5" library="Разъёмы штырьковые 2.54мм" package="2X14" value="" x="-92.71" y="16.51"/>
 </elements>
 <signals>
