File: reversator/reversator.sch (EAGLE design)
At the start: 6 parts

Commit message: 2
Parts:
- added U$1: 1X8, headers(2mm):1X8
Changed lines of the file:
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@@
 <setting verticaltext="up"/>
 </settings>
-<grid distance="100" unitdist="mil" unit="mil" style="lines" multiple="1" display="yes" altdistance="0.01" altunitdist="inch" altunit="inch"/>
+<grid distance="0.1" unitdist="inch" unit="inch" style="lines" multiple="1" display="yes" altdistance="0.01" altunitdist="inch" altunit="inch"/>
 <layers>
 <layer number="1" name="Top" color="4" fill="1" visible="no" active="no"/>
@@
 <part name="C72" library="h1,27mm" deviceset="1X54" device=""/>
 <part name="C60" library="h1,27mm" deviceset="1X54" device=""/>
+<part name="U$1" library="headers(2mm)" deviceset="1X8" device=""/>
 </parts>
 <sheets>
@@
 <instance part="C72" gate="G$1" x="241.3" y="330.2" rot="MR180"/>
 <instance part="C60" gate="G$1" x="205.74" y="327.66"/>
+<instance part="U$1" gate="G$1" x="104.14" y="345.44"/>
 </instances>
 <busses>
@@
 </segment>
 </bus>
-<bus name="A[0..15],D[0..7],PA[0..13],!PA13,PD[0..7],CLK21,CLK26,CLK_P21,CLK_P26,CIRAM-A10,CIRAM-CS,!IRQ,M2,!NMI,PALE,!PPU,!PRD,!PWE,!RAM,!ROMSEL,R/!W,!RST21,!RST26,!RST_P21,!RST_P26,4016CUP,4016RD_!OE,4016WR_B[0..2],4016RD_D[0..4],4017CUP,4017RD_!OE,4017RD_D[0..4],VIDEO21,VIDEO26,MIC,SND_IN,SND_OUT,SOUND21_[1..2],SOUND21,SOUND26_[1..2],SOUND26">
-<segment>
-<wire x1="185.42" y1="261.62" x2="185.42" y2="396.24" width="0.762" layer="92"/>
-</segment>
-</bus>

Commit message: .
Parts:
- removed U$1: 1X8, headers(2mm):1X8
- added JP2, JP3, JP4, JP5: (no value), Разъёмы штырьковые 2.54мм:PINHD-2X14
Changed lines of the file:
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@@
 <part name="C72" library="h1,27mm" deviceset="1X54" device=""/>
 <part name="C60" library="h1,27mm" deviceset="1X54" device=""/>
-<part name="U$1" library="headers(2mm)" deviceset="1X8" device=""/>
+<part name="JP2" library="Разъёмы штырьковые 2.54мм" deviceset="PINHD-2X14" device=""/>
+<part name="JP3" library="Разъёмы штырьковые 2.54мм" deviceset="PINHD-2X14" device=""/>
+<part name="JP4" library="Разъёмы штырьковые 2.54мм" deviceset="PINHD-2X14" device=""/>
+<part name="JP5" library="Разъёмы штырьковые 2.54мм" deviceset="PINHD-2X14" device=""/>
 </parts>
 <sheets>
@@
 <instance part="C72" gate="G$1" x="241.3" y="330.2" rot="MR180"/>
 <instance part="C60" gate="G$1" x="205.74" y="327.66"/>
-<instance part="U$1" gate="G$1" x="104.14" y="345.44"/>
+<instance part="JP2" gate="A" x="66.04" y="304.8"/>
+<instance part="JP3" gate="A" x="109.22" y="307.34"/>
+<instance part="JP4" gate="A" x="66.04" y="256.54"/>
+<instance part="JP5" gate="A" x="114.3" y="256.54"/>
 </instances>
 <busses>
